Commit message: Add `gazebo_launch.py` and update robot model [2.2]

File: src/dribot_description/urdf/dribot_description.xacro (robot description, xacro)
@@ -41,3 +41,23 @@
   <xacro:caster prefix="caster_rear" x_pos="${-base_to_caster}"
                 radius="${(wheel_radius+wheel_zoff-(base_height/2))}"/>
+  <gazebo>
+    <plugin name='diff_drive' filename='libgazebo_ros_diff_drive.so'>
+      <!-- Make sure the names here match joints specified in our wheel.xacro
+           in case of our code they are named `{prefix}_joint`, where prefix
+           is declared when we call xacro:wheel. -->
+      <left_joint>wheel_left_joint</left_joint>
+      <right_joint>wheel_right_joint</right_joint>
+      <!-- In the two lines below we are using parameters to calculate values
+           that we pass into the plugin. -->
+      <wheel_separation>${2*base_radius+2*wheel_ygap+2*wheel_width/2}</wheel_separation>
+      <wheel_diameter>${2*wheel_radius}</wheel_diameter>
+      <max_wheel_torque>20</max_wheel_torque>
+      <max_wheel_acceleration>1.0</max_wheel_acceleration>
+      <publish_odom>true</publish_odom>
+      <publish_odom_tf>true</publish_odom_tf>
+      <publish_wheel_tf>true</publish_wheel_tf>
+      <odometry_frame>odom</odometry_frame>
+      <robot_base_frame>base_link</robot_base_frame>
+    </plugin>
+  </gazebo>
 </robot>

File: src/dribot_description/urdf/wheel.xacro (robot description, xacro)
@@ -23,4 +23,12 @@
       <axis xyz="0 1 0"/>
     </joint>
+    <gazebo reference="${prefix}_link">
+      <mu1 value="0.50"/>
+      <mu2 value="3.0"/>
+      <kp  value="10000000.0" />
+      <kd  value="100.0" />
+      <fdir1 value="0 0 1"/>
+      <material>Gazebo/Black</material>
+    </gazebo>
   </xacro:macro>
 </robot>
